File: PCB/keyboard.kicad_pcb (KiCad board)
At the start: 2 copper layers, 350.8 x 138.6 mm, 167 parts, among them J1 OLED_128x32, SW1 RotaryEncoder_Switch, U1 Raspberry_Pi_Pico

Commit message: Add files via upload
Routing:
- net Row 3: track 278.6 -> 416.0 mm
- net GND: track 448.9 -> 470.3 mm, vias 6 -> 7
Changed lines of the file:
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@@
+	)
+	(segment
+		(start -13.119 48.599)
+		(end -20.739 40.979)
+		(width 0.2)
+		(layer "F.Cu")
+		(net 34)
+	)
+	(segment
+		(start -24.841 61.061)
+		(end -19.239 61.061)
+		(width 0.2)
+		(layer "F.Cu")
+		(net 34)
+	)
+	(segment
+		(start 13.058924 97.819)
+		(end 23.044924 107.805)
+		(width 0.2)
+		(layer "F.Cu")
+		(net 34)
+	)
+	(segment
+		(start 8.669057 97.819)
+		(end 13.058924 97.819)
+		(width 0.2)
+		(layer "F.Cu")
+		(net 34)
+	)
+	(segment
+		(start -19.239 61.061)
+		(end -14.151 66.149)
+		(width 0.2)
+		(layer "F.Cu")
+		(net 34)
+	)
+	(segment
+		(start 23.044924 107.805)
+		(end 26.19375 107.805)
+		(width 0.2)
+		(layer "F.Cu")
+		(net 34)
+	)
+	(segment
+		(start -25.242 60.66)
+		(end -24.841 61.061)
+		(width 0.2)
+		(layer "F.Cu")
+		(net 34)
 	)
 	(segment
 		(start 26.19375 107.805)
 		(end 304.8 107.805)
+		(width 0.2)
+		(layer "F.Cu")
+		(net 34)
+	)
+	(segment
+		(start -4.11 54.83)
+		(end 2.652957 54.83)
+		(width 0.2)
+		(layer "F.Cu")
+		(net 34)
+	)
+	(segment
+		(start -24.841 40.979)
+		(end -25.242 41.38)
+		(width 0.2)
+		(layer "F.Cu")
+		(net 34)
+	)
+	(segment
+		(start -25.242 41.38)
+		(end -25.242 60.66)
+		(width 0.2)
+		(layer "F.Cu")
+		(net 34)
+	)
+	(segment
+		(start -20.739 40.979)
+		(end -24.841 40.979)
+		(width 0.2)
+		(layer "F.Cu")
+		(net 34)
+	)
+	(segment
+		(start -14.151 66.149)
+		(end -14.151 74.998943)
+		(width 0.2)
+		(layer "F.Cu")
+		(net 34)
+	)
+	(segment
+		(start 2.652957 52.410957)
+		(end -1.159 48.599)
+		(width 0.2)
+		(layer "F.Cu")
+		(net 34)
+	)
+	(segment
+		(start -1.159 48.599)
+		(end -13.119 48.599)
+		(width 0.2)
+		(layer "F.Cu")
+		(net 34)
+	)
+	(segment
+		(start 2.652957 54.83)
+		(end 2.652957 52.410957)
+		(width 0.2)
+		(layer "F.Cu")
+		(net 34)
+	)
+	(segment
+		(start -14.151 74.998943)
+		(end 8.669057 97.819)
 		(width 0.2)
 		(layer "F.Cu")
@@
 	)
 	(segment
+		(start -24.841 35.661)
+		(end -23.452 37.05)
+		(width 0.2)
+		(layer "F.Cu")
+		(net 91)
+	)
+	(segment
 		(start 279.6 31.2)
 		(end 279.6 46.79)
@@
 	)
 	(segment
+		(start -23.452 37.05)
+		(end -21.89 37.05)
+		(width 0.2)
+		(layer "F.Cu")
+		(net 91)
+	)
+	(segment
 		(start -21.14 61.7)
 		(end -21.89 62.45)
@@
 	)
 	(segment
-		(start -22.262002 38.239998)
-		(end -24.841 35.661)
-		(width 0.2)
-		(layer "F.Cu")
-		(net 91)
-	)
-	(segment
 		(start 1.7 57.2)
 		(end 3.9725 54.9275)
@@
 	)
 	(segment
+		(start -17.649 37.05)
+		(end -6.7 47.999)
+		(width 0.2)
+		(layer "F.Cu")
+		(net 91)
+	)
+	(segment
 		(start 314.325 28.8)
 		(end 317.0375 26.0875)
@@
 	)
 	(segment
-		(start -21.902385 38.239998)
-		(end -21.89 38.227613)
-		(width 0.2)
-		(layer "F.Cu")
-		(net 91)
-	)
-	(segment
 		(start -17 65.2)
 		(end -20.5 61.7)
@@
 	)
 	(segment
-		(start -21.902385 38.239998)
-		(end -22.262002 38.239998)
-		(width 0.2)
-		(layer "F.Cu")
-		(net 91)
-	)
-	(segment
 		(start -5.9 57.1)
 		(end -5.9 51.54)
@@
 	)
 	(segment
-		(start -21.89 38.227613)
-		(end -21.89 37.05)
-		(width 0.2)
-		(layer "F.Cu")
-		(net 91)
-	)
-	(segment
 		(start -15.7 23.4)
 		(end -14.75 24.35)
@@
 		(start 3.9725 54.9275)
 		(end 271.4625 54.9275)
+		(width 0.2)
+		(layer "F.Cu")
+		(net 91)
+	)
+	(segment
+		(start -21.89 37.05)
+		(end -17.649 37.05)
 		(width 0.2)
 		(layer "F.Cu")
@@
 	)
 	(via
+		(at -6.7 47.999)
+		(size 0.6)
+		(drill 0.3)
+		(layers "F.Cu" "B.Cu")
+		(net 91)
+	)
+	(via
 		(at 279.6 31.2)
 		(size 0.6)
@@
 	)
 	(segment
+		(start -4.949 49.75)
+		(end -4.11 49.75)
+		(width 0.2)
+		(layer "B.Cu")
+		(net 91)
+	)
+	(segment
 		(start -5.9 57.46853)
 		(end -5.9 58.3)
@@
 		(width 0.2)
 		(layer "B.Cu")
+		(net 91)
+	)
+	(segment
+		(start -6.7 47.999)
+		(end -4.949 49.75)
+		(width 0.2)
+		(layer "B.Cu")

Commit message: Add files via upload
Parts:
- moved J1 24.7 mm to (260.5, 22.3)
Connections:
- U1 pad 36: unconnected-(U1-3V3-Pad36) -> OLED 3V3
- U1 pad 37: OLED 3V3 -> unconnected-(U1-3V3_EN-Pad37)
Routing:
- net OLED SDA: track 291.6 -> 598.9 mm, vias 1 -> 0
- net OLED 3V3: track 346.9 -> 275.1 mm, vias 4 -> 1
- net OLED SCL: track 459.1 -> 403.8 mm
- net GND: track 470.3 -> 486.9 mm, vias 7 -> 4
- removed copper zone on B.Cu, net (none)
- removed copper zone on F.Cu, net (none)

Commit message: Add files via upload
Parts:
- added D84: Diode, ScottoKeebs_Components:Diode_DO-35, B.Cu at (-5.50, 102.5)
- added D85: Diode, ScottoKeebs_Components:Diode_DO-35, B.Cu at (-5.40, 121.1)
- added D86: Diode, ScottoKeebs_Components:Diode_DO-35, B.Cu at (-5.40, 140.2)
- added S84: Keyswitch, ScottoKeebs_Hotswap:Hotswap_MX_1.00u, F.Cu at (-14.9, 98.1)
- added S85: Keyswitch, ScottoKeebs_Hotswap:Hotswap_MX_1.00u, F.Cu at (-14.9, 117.2)
- added S86: Keyswitch, ScottoKeebs_Hotswap:Hotswap_MX_1.00u, F.Cu at (-14.9, 136.2)
- U1: value Raspberry_Pi_Pico -> ESP32-S3-DevKitC; footprint ScottoKeebs_MCU:Raspberry_Pi_Pico -> PCM_Espressif:ESP32-S3-DevKitC
- moved J1 133.0 mm to (127.5, 22.8)
- moved U1 26.0 mm to (-23.9, 19.8)
- moved SW1 15.7 mm to (286.9, 24.3)
Connections:
- U1 pad 1: Column 1 -> OLED 3V3
- U1 pad 10: Column 8 -> Column 15
- U1 pad 11: Column 9 -> Row 0
- U1 pad 12: Column 10 -> Column 8
- U1 pad 13: GND -> Column 3
- U1 pad 14: Column 11 -> RotaryRight
- U1 pad 15: Column 12 -> Column 9
- U1 pad 16: Column 13 -> Column 10
- U1 pad 17: Row 0 -> Column 11
- U1 pad 18: GND -> Column 12
- U1 pad 19: Row 1 -> Column 13
- U1 pad 2: Column 2 -> OLED 3V3
- U1 pad 20: Row 2 -> Column 14
- U1 pad 21: OLED SDA -> unconnected-(U1-5V-Pad21)
- U1 pad 22: OLED SCL -> GND
- U1 pad 24: Row 5 -> GND
- U1 pad 25: Row 4 -> unconnected-(U1-GPIO19/USB_D--Pad25)
- U1 pad 26: Row 3 -> unconnected-(U1-GPIO20/USB_D+-Pad26)
- U1 pad 27: RotaryLeft -> Row 1
- U1 pad 28: GND -> RotaryLeft
- U1 pad 29: RotaryRight -> unconnected-(U1-GPIO48-Pad29)
- U1 pad 3: GND -> unconnected-(U1-CHIP_PU-Pad3)
- U1 pad 30: unconnected-(U1-RUN-Pad30) -> RotaryClick
- U1 pad 31: RotaryClick -> Column 0
- U1 pad 32: Column 0 -> Row 2
- U1 pad 33: unconnected-(U1-AGND-Pad33) -> Row 3
- U1 pad 34: Column 14 -> Row 4
- U1 pad 35: unconnected-(U1-ADC_VREF-Pad35) -> Row 5
- U1 pad 36: OLED 3V3 -> unconnected-(U1-GPIO39/MTCK-Pad36)
- U1 pad 38: GND -> unconnected-(U1-GPIO41/MTDI-Pad38)
- U1 pad 4: Column 3 -> Column 4
- U1 pad 40: unconnected-(U1-VBUS-Pad40) -> Column 2
- U1 pad 41: unconnected-(U1-SWCLK-Pad41) -> Column 1
- U1 pad 5: Column 4 -> Column 5
- U1 pad 6: Column 5 -> Column 6
- U1 pad 7: Column 6 -> Column 7
- U1 pad 8: GND -> OLED SDA
- U1 pad 9: Column 7 -> OLED SCL
Routing:
- net OLED SDA: track 598.9 -> 166.4 mm, vias 0 -> 6
- net OLED SCL: track 403.8 -> 170.5 mm, vias 1 -> 4
- net Row 1: track 493.7 -> 309.2 mm
- net Column 13: track 475.4 -> 328.2 mm, vias 1 -> 3
- net Column 12: track 520.1 -> 376.4 mm, vias 0 -> 3
- net Column 9: track 443.8 -> 314.2 mm, vias 1 -> 3
- net Column 10: track 461.5 -> 332.4 mm, vias 0 -> 2
- net Row 2: track 451.8 -> 339.5 mm, vias 0 -> 1
- net OLED 3V3: track 275.1 -> 162.8 mm, vias 1 -> 2
- net GND: track 486.9 -> 393.2 mm
- net Column 15: track 0.00 -> 93.0 mm
- net Column 11: track 488.1 -> 397.2 mm, vias 0 -> 3
- net Column 14: track 550.4 -> 473.1 mm, vias 0 -> 3
- net Column 0: track 154.8 -> 107.8 mm
- net Row 3: track 416.0 -> 370.3 mm, vias 0 -> 2
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Other:
- board size 350.8 x 138.6 mm -> 337.6 x 138.6 mm

Commit message: Add files via upload
Other:
- board size 337.6 x 138.6 mm -> 334.6 x 136.8 mm
Changed lines of the file:
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@@
 	(gr_rect
 		(start -26.5 17.6)
-		(end 311.1 156.2)
+		(end 308.1 154.4)
 		(stroke
 			(width 0.05)

Commit message: Add kicad files
Parts:
- removed D84, D85, D86: Diode, ScottoKeebs_Components:Diode_DO-35
- removed S84, S85, S86: Keyswitch, ScottoKeebs_Hotswap:Hotswap_MX_1.00u
- added D83: Diode, ScottoKeebs_Components:Diode_DO-35, B.Cu at (-3.30, 142.1)
- added S83: Keyswitch, ScottoKeebs_Hotswap:Hotswap_MX_1.00u, F.Cu at (-12.8, 138.2)
- S27, S69: footprint ScottoKeebs_Hotswap:Hotswap_MX_1.00u -> ScottoKeebs_Hotswap:Hotswap_MX_2.00u
- S29: footprint ScottoKeebs_Hotswap:Hotswap_MX_2.00u -> ScottoKeebs_Hotswap:Hotswap_MX_1.50u
- S37: footprint ScottoKeebs_Hotswap:Hotswap_MX_1.75u -> ScottoKeebs_Hotswap:Hotswap_MX_1.00u
- S39: footprint ScottoKeebs_Hotswap:Hotswap_MX_1.50u -> ScottoKeebs_Hotswap:Hotswap_MX_1.00u
- S42: footprint ScottoKeebs_Hotswap:Hotswap_MX_1.00u -> ScottoKeebs_Hotswap:Hotswap_MX_1.50u
- S44: footprint ScottoKeebs_Hotswap:Hotswap_MX_1.00u -> ScottoKeebs_Hotswap:Hotswap_MX_1.75u
- S51, S66: footprint ScottoKeebs_Hotswap:Hotswap_MX_2.00u -> ScottoKeebs_Hotswap:Hotswap_MX_1.00u
- S53: footprint ScottoKeebs_Hotswap:Hotswap_MX_2.25u -> ScottoKeebs_Hotswap:Hotswap_MX_1.00u
- S56: footprint ScottoKeebs_Hotswap:Hotswap_MX_1.00u -> ScottoKeebs_Hotswap:Hotswap_MX_2.25u
- S58: footprint ScottoKeebs_Hotswap:Hotswap_MX_1.50u -> ScottoKeebs_Hotswap:Hotswap_MX_2.00u
- S60: footprint ScottoKeebs_Hotswap:Hotswap_MX_6.25u -> ScottoKeebs_Hotswap:Hotswap_MX_1.00u
- S61, S62, S63: footprint ScottoKeebs_Hotswap:Hotswap_MX_1.25u -> ScottoKeebs_Hotswap:Hotswap_MX_1.00u
- S72, S73, S74: footprint ScottoKeebs_Hotswap:Hotswap_MX_1.00u -> ScottoKeebs_Hotswap:Hotswap_MX_1.25u
- S75: footprint ScottoKeebs_Hotswap:Hotswap_MX_1.00u -> ScottoKeebs_Hotswap:Hotswap_MX_6.25u
- moved D82 309.8 mm to (-4.20, 123.0)
- moved S82 309.0 mm to (-12.8, 119.1)
- moved D72 282.2 mm to (23.2, 146.2)
- moved S72 282.2 mm to (13.7, 142.4)
- moved D29 279.9 mm to (25.6, 89.1)
- moved S29 279.8 mm to (16.0, 85.2)
- moved D44 277.5 mm to (28.0, 108.1)
- moved S44 277.5 mm to (18.4, 104.3)
- moved D58 275.1 mm to (30.4, 127.2)
- moved S58 275.1 mm to (20.8, 123.3)
- moved D14 246.6 mm to (20.9, 70.0)
- moved S14 246.6 mm to (11.3, 66.2)
- moved J1 124.3 mm to (250.8, 38.1)
- moved D75 73.2 mm to (142.3, 146.2)
- moved S75 73.2 mm to (132.7, 142.4)
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Connections:
- D14 pad 1: Row 0 -> Row 1
- D29 pad 1: Row 1 -> Row 2
- D44 pad 1: Row 2 -> Row 3
- D58 pad 1: Row 3 -> Row 4
- D72 pad 1: Row 4 -> Row 5
- D82 pad 1: Row 5 -> Row 4
- S14 pad 1: Column 13 -> Column 0
- S15 pad 1: Column 0 -> Column 1
- S16 pad 1: Column 1 -> Column 2
- S17 pad 1: Column 2 -> Column 3
- S18 pad 1: Column 3 -> Column 4
- S19 pad 1: Column 4 -> Column 5
- S20 pad 1: Column 5 -> Column 6
- S21 pad 1: Column 6 -> Column 7
- S22 pad 1: Column 7 -> Column 8
- S23 pad 1: Column 8 -> Column 9
- S24 pad 1: Column 9 -> Column 10
- S25 pad 1: Column 10 -> Column 11
- S26 pad 1: Column 11 -> Column 12
- S27 pad 1: Column 12 -> Column 13
- S28 pad 1: Column 13 -> Column 14
- S29 pad 1: Column 14 -> Column 0
- S30 pad 1: Column 0 -> Column 1
- S31 pad 1: Column 1 -> Column 2
- S32 pad 1: Column 2 -> Column 3
- S33 pad 1: Column 3 -> Column 4
- S34 pad 1: Column 4 -> Column 5
- S35 pad 1: Column 5 -> Column 6
- S36 pad 1: Column 6 -> Column 7
- S37 pad 1: Column 7 -> Column 8
- S38 pad 1: Column 8 -> Column 9
- S39 pad 1: Column 9 -> Column 10
- S40 pad 1: Column 10 -> Column 11
- S41 pad 1: Column 11 -> Column 12
- S42 pad 1: Column 12 -> Column 13
- S43 pad 1: Column 13 -> Column 14
- S44 pad 1: Column 14 -> Column 0
- S45 pad 1: Column 0 -> Column 1
- S46 pad 1: Column 1 -> Column 2
- S47 pad 1: Column 2 -> Column 3
- S48 pad 1: Column 3 -> Column 4
- S49 pad 1: Column 4 -> Column 5
- S50 pad 1: Column 5 -> Column 6
- S51 pad 1: Column 6 -> Column 7
- S52 pad 1: Column 7 -> Column 8
- S53 pad 1: Column 8 -> Column 9
- S54 pad 1: Column 9 -> Column 10
- S55 pad 1: Column 10 -> Column 11
- S56 pad 1: Column 11 -> Column 12
- S57 pad 1: Column 12 -> Column 14
- S58 pad 1: Column 14 -> Column 0
- S59 pad 1: Column 0 -> Column 1
- S60 pad 1: Column 1 -> Column 2
- S61 pad 1: Column 2 -> Column 3
- S62 pad 1: Column 3 -> Column 4
- S63 pad 1: Column 4 -> Column 5
- S64 pad 1: Column 5 -> Column 6
- S65 pad 1: Column 6 -> Column 7
- S66 pad 1: Column 7 -> Column 8
- S67 pad 1: Column 8 -> Column 9
- S68 pad 1: Column 9 -> Column 10
- S69 pad 1: Column 10 -> Column 11
- S70 pad 1: Column 11 -> Column 12
- S71 pad 1: Column 12 -> Column 14
- S72 pad 1: Column 14 -> Column 0
- S73 pad 1: Column 0 -> Column 1
- S74 pad 1: Column 1 -> Column 2
- S75 pad 1: Column 2 -> Column 5
- S76 pad 1: Column 5 -> Column 8
- S77 pad 1: Column 8 -> Column 9
- S78 pad 1: Column 9 -> Column 10
- S79 pad 1: Column 10 -> Column 11
- S80 pad 1: Column 11 -> Column 12
- S81 pad 1: Column 12 -> Column 14
- S82 pad 1: Column 14 -> Column 15
Routing:
- net OLED SCL: track 170.5 -> 304.9 mm, vias 4 -> 5
- net OLED SDA: track 166.4 -> 299.4 mm
- net OLED 3V3: track 162.8 -> 291.2 mm, vias 2 -> 9
- net Column 14: track 473.1 -> 425.4 mm, vias 3 -> 5
- net Column 8: track 297.0 -> 328.1 mm, vias 1 -> 11
- net Column 9: track 314.2 -> 339.8 mm, vias 3 -> 11
- net Column 0: track 107.8 -> 131.3 mm, vias 1 -> 7
- net Column 2: track 154.0 -> 175.8 mm, vias 1 -> 11
- net Row 3: track 370.3 -> 348.5 mm
- net Column 3: track 202.5 -> 182.0 mm, vias 3 -> 7
- net Column 12: track 376.4 -> 396.7 mm, vias 3 -> 8
- net Column 10: track 332.4 -> 352.4 mm, vias 2 -> 8
- net RotaryLeft: track 325.5 -> 345.0 mm, vias 2 -> 4
- net RotaryClick: track 318.0 -> 337.3 mm, vias 2 -> 1
- net Row 2: track 339.5 -> 326.5 mm, vias 1 -> 2
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Other:
- board size 334.6 x 136.8 mm -> 335.4 x 118.1 mm
- board text added: "HackClub"
- board text added: "Haft"
- board text added: "Highway to UnderCity"
