File: PCB/keyboard.kicad_sch (KiCad schematic)
At the start: 167 parts, among them J1 OLED_128x32, SW1 RotaryEncoder_Switch, U1 Raspberry_Pi_Pico

Commit message: Add files via upload
Connections:
- net OLED 3V3: now also U1.36 (3V3); no longer U1.37 (3V3_EN)
Changed lines of the file:
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@@
 	(global_label "OLED 3V3"
 		(shape input)
-		(at 73.66 33.02 0)
+		(at 73.66 35.56 0)
 		(fields_autoplaced yes)
 		(effects
@@
 		)
 		(property "Intersheetrefs" "${INTERSHEET_REFS}"
-			(at 85.898 33.02 0)
+			(at 85.898 35.56 0)
 			(effects
 				(font

Commit message: Add files via upload
Parts:
- removed U1: Raspberry_Pi_Pico, ScottoKeebs_MCU:Raspberry_Pi_Pico, symbol ScottoKeebs:MCU_Raspberry_Pi_Pico
- added D84, D85, D86: Diode, ScottoKeebs_Components:Diode_DO-35, symbol ScottoKeebs:Placeholder_Diode
- added S84, S85, S86: Keyswitch, ScottoKeebs_Hotswap:Hotswap_MX_1.00u, symbol ScottoKeebs:Placeholder_Keyswitch
- added U1: ESP32-S3-DevKitC, PCM_Espressif:ESP32-S3-DevKitC, symbol PCM_Espressif:ESP32-S3-DevKitC
Connections:
- net Column 0: now also U1.31 (GPIO0)
- net Column 1: now also U1.41 (GPIO1/ADC1_CH0)
- net Column 10: now also U1.16 (GPIO10/ADC1_CH9)
- net Column 11: now also U1.17 (GPIO11/ADC2_CH0)
- net Column 12: now also U1.18 (GPIO12/ADC2_CH1)
- net Column 13: now also U1.19 (GPIO13/ADC2_CH2)
- net Column 14: now also U1.20 (GPIO14/ADC2_CH3)
- net Column 2: now also U1.40 (GPIO2/ADC1_CH1)
- net Column 3: now also U1.13 (GPIO3/ADC1_CH2)
- net Column 4: now also U1.4 (GPIO4/ADC1_CH3)
- net Column 5: now also U1.5 (GPIO5/ADC1_CH4)
- net Column 6: now also U1.6 (GPIO6/ADC1_CH5)
- net Column 7: now also U1.7 (GPIO7/ADC1_CH6)
- net Column 8: now also U1.12 (GPIO8/ADC1_CH7)
- net Column 9: now also U1.15 (GPIO9/ADC1_CH8)
- net GND: now also U1.22 (GND), U1.23 (GND), U1.24 (GND), U1.44 (GND)
- net OLED 3V3: now also U1.1 (3V3), U1.2 (3V3)
- net OLED SCL: now also U1.9 (GPIO16/ADC2_CH5/32K_N)
- net OLED SDA: now also U1.8 (GPIO15/ADC2_CH4/32K_P)
- net RotaryClick: now also U1.30 (GPIO45)
- net RotaryLeft: now also U1.28 (GPIO47)
- net RotaryRight: now also U1.14 (GPIO46)
- net Row 0: now also U1.11 (GPIO18/ADC2_CH7)
- net Row 1: now also U1.27 (GPIO21)
- net Row 2: now also U1.32 (GPIO35)
- net Row 3: now also D84.1 (K), U1.33 (GPIO36)
- net Row 4: now also D85.1 (K), U1.34 (GPIO37)
- net Row 5: now also D86.1 (K), U1.35 (GPIO38)
- new net: D84.2 (A), S84.2
- new net: D85.2 (A), S85.2
- new net: D86.2 (A), S86.2
- new net Column 15: S84.1, S85.1, S86.1, U1.10 (GPIO17/ADC2_CH6)

Commit message: Add kicad files
Parts:
- removed D14, D84: Diode, ScottoKeebs_Components:Diode_DO-35, symbol ScottoKeebs:Placeholder_Diode
- removed S14, S84: Keyswitch, ScottoKeebs_Hotswap:Hotswap_MX_1.00u, symbol ScottoKeebs:Placeholder_Keyswitch
- S27: renamed from S28; footprint ScottoKeebs_Hotswap:Hotswap_MX_1.00u -> ScottoKeebs_Hotswap:Hotswap_MX_2.00u
- S28: renamed from S29; footprint ScottoKeebs_Hotswap:Hotswap_MX_2.00u -> ScottoKeebs_Hotswap:Hotswap_MX_1.00u
- S29: renamed from S30; footprint ScottoKeebs_Hotswap:Hotswap_MX_1.00u -> ScottoKeebs_Hotswap:Hotswap_MX_1.50u
- S36: renamed from S37; footprint ScottoKeebs_Hotswap:Hotswap_MX_1.75u -> ScottoKeebs_Hotswap:Hotswap_MX_1.00u
- S38: renamed from S39; footprint ScottoKeebs_Hotswap:Hotswap_MX_1.50u -> ScottoKeebs_Hotswap:Hotswap_MX_1.00u
- S42: renamed from S43; footprint ScottoKeebs_Hotswap:Hotswap_MX_1.00u -> ScottoKeebs_Hotswap:Hotswap_MX_1.50u
- S44: renamed from S45; footprint ScottoKeebs_Hotswap:Hotswap_MX_1.00u -> ScottoKeebs_Hotswap:Hotswap_MX_1.75u
- S50: renamed from S51; footprint ScottoKeebs_Hotswap:Hotswap_MX_2.00u -> ScottoKeebs_Hotswap:Hotswap_MX_1.00u
- S52: renamed from S53; footprint ScottoKeebs_Hotswap:Hotswap_MX_2.25u -> ScottoKeebs_Hotswap:Hotswap_MX_1.00u
- S56: renamed from S57; footprint ScottoKeebs_Hotswap:Hotswap_MX_1.00u -> ScottoKeebs_Hotswap:Hotswap_MX_2.25u
- S57: renamed from S58; footprint ScottoKeebs_Hotswap:Hotswap_MX_1.50u -> ScottoKeebs_Hotswap:Hotswap_MX_1.00u
- S58: renamed from S59; footprint ScottoKeebs_Hotswap:Hotswap_MX_1.00u -> ScottoKeebs_Hotswap:Hotswap_MX_2.00u
- S59: renamed from S60; footprint ScottoKeebs_Hotswap:Hotswap_MX_6.25u -> ScottoKeebs_Hotswap:Hotswap_MX_1.00u
- S60: renamed from S61; footprint ScottoKeebs_Hotswap:Hotswap_MX_1.25u -> ScottoKeebs_Hotswap:Hotswap_MX_1.00u
- S61: renamed from S62; footprint ScottoKeebs_Hotswap:Hotswap_MX_1.25u -> ScottoKeebs_Hotswap:Hotswap_MX_1.00u
- S62: renamed from S63; footprint ScottoKeebs_Hotswap:Hotswap_MX_1.25u -> ScottoKeebs_Hotswap:Hotswap_MX_1.00u
- S65: renamed from S66; footprint ScottoKeebs_Hotswap:Hotswap_MX_2.00u -> ScottoKeebs_Hotswap:Hotswap_MX_1.00u
- S69: renamed from S70; footprint ScottoKeebs_Hotswap:Hotswap_MX_1.00u -> ScottoKeebs_Hotswap:Hotswap_MX_2.00u
- S72: renamed from S73; footprint ScottoKeebs_Hotswap:Hotswap_MX_1.00u -> ScottoKeebs_Hotswap:Hotswap_MX_1.25u
- S73: renamed from S74; footprint ScottoKeebs_Hotswap:Hotswap_MX_1.00u -> ScottoKeebs_Hotswap:Hotswap_MX_1.25u
- S74: renamed from S75; footprint ScottoKeebs_Hotswap:Hotswap_MX_1.00u -> ScottoKeebs_Hotswap:Hotswap_MX_1.25u
- S75: renamed from S76; footprint ScottoKeebs_Hotswap:Hotswap_MX_1.00u -> ScottoKeebs_Hotswap:Hotswap_MX_6.25u
- renumbered D15 to D14, D16 to D15, D17 to D16, D18 to D17, D19 to D18, D20 to D19, D21 to D20, D22 to D21, D23 to D22, D24 to D23, D25 to D24, D26 to D25, D27 to D26, D28 to D27, D29 to D28, D30 to D29, D31 to D30, D32 to D31, D33 to D32, D34 to D33, D35 to D34, D36 to D35, D37 to D36, D38 to D37, D39 to D38, D40 to D39, D41 to D40, D42 to D41, D43 to D42, D44 to D43, D45 to D44, D46 to D45, D47 to D46, D48 to D47, D49 to D48, D50 to D49, D51 to D50, D52 to D51, D53 to D52, D54 to D53, D55 to D54, D56 to D55, D57 to D56, D58 to D57, D59 to D58, D60 to D59, D61 to D60, D62 to D61, D63 to D62, D64 to D63, D65 to D64, D66 to D65, D67 to D66, D68 to D67, D69 to D68, D70 to D69, D71 to D70, D72 to D71, D73 to D72, D74 to D73, D75 to D74, D76 to D75, D77 to D76, D78 to D77, D79 to D78, D80 to D79, D81 to D80, D82 to D81, D85 to D82, D86 to D83, S15 to S14, S16 to S15, S17 to S16, S18 to S17, S19 to S18, S20 to S19, S21 to S20, S22 to S21, S23 to S22, S24 to S23, S25 to S24, S26 to S25, S27 to S26, S31 to S30, S32 to S31, S33 to S32, S34 to S33, S35 to S34, S36 to S35, S38 to S37, S40 to S39, S41 to S40, S42 to S41, S44 to S43, S46 to S45, S47 to S46, S48 to S47, S49 to S48, S50 to S49, S52 to S51, S54 to S53, S55 to S54, S56 to S55, S64 to S63, S65 to S64, S67 to S66, S68 to S67, S69 to S68, S71 to S70, S72 to S71, S77 to S76, S78 to S77, S79 to S78, S80 to S79, S81 to S80, S82 to S81, S85 to S82, S86 to S83
